File: ActiveSplitterPedal/SOT23/ActiveSplitterPedal_SOT23.kicad_pcb (KiCad board)
At the start: 2 copper layers, 48 parts, among them J1 MonoJack2Switch, J2 MonoJack2Switch, J3 MonoJack2Switch, J4 MonoJack2Switch, J5 MonoJack2Switch, J6 Barrel_Jack, SW1 SW_DIP_x04, U1 OPA842, U10 TPS60400, U2 OPA842, U3 OPA842, U4 OPA842, U5 DG468DV_T1_E3, U6 DG468DV_T1_E3, U7 DG468DV_T1_E3, U8 DG468DV_T1_E3, U9 SE8250X2

Commit message: updated schematic
Parts:
- added R10: 100R, Resistor_SMD:R_0805_2012Metric_Pad1.15x1.40mm_HandSolder, B.Cu at (110.7, 129.9)
- added R11: 2K2, Resistor_SMD:R_0805_2012Metric_Pad1.15x1.40mm_HandSolder, B.Cu at (111.8, 107.8)
- added R12: 100R, Resistor_SMD:R_0805_2012Metric_Pad1.15x1.40mm_HandSolder, B.Cu at (106.0, 132.8)
- added R13: 2K2, Resistor_SMD:R_0805_2012Metric_Pad1.15x1.40mm_HandSolder, B.Cu at (111.4, 85.5)
- added R14: 100R, Resistor_SMD:R_0805_2012Metric_Pad1.15x1.40mm_HandSolder, B.Cu at (111.8, 104.9)
- added R15: 2K2, Resistor_SMD:R_0805_2012Metric_Pad1.15x1.40mm_HandSolder, B.Cu at (104.1, 57.2)
- added R16: 100R, Resistor_SMD:R_0805_2012Metric_Pad1.15x1.40mm_HandSolder, B.Cu at (107.0, 107.8)
- added R17: 100R, Resistor_SMD:R_0805_2012Metric_Pad1.15x1.40mm_HandSolder, B.Cu at (111.4, 82.6)
- added R18: 100R, Resistor_SMD:R_0805_2012Metric_Pad1.15x1.40mm_HandSolder, B.Cu at (106.7, 85.5)
- added R19: 100R, Resistor_SMD:R_0805_2012Metric_Pad1.15x1.40mm_HandSolder, B.Cu at (104.1, 60.2)
- added R20: 100R, Resistor_SMD:R_0805_2012Metric_Pad1.15x1.40mm_HandSolder, B.Cu at (108.8, 57.2)
- added R9: 2K2, Resistor_SMD:R_0805_2012Metric_Pad1.15x1.40mm_HandSolder, B.Cu at (110.7, 132.8)
- added RV1: 5K, Potentiometer_THT:Potentiometer_Alps_RK09L_Single_Vertical, F.Cu at (116.5, 60.3)
- added RV2: 5K, Potentiometer_THT:Potentiometer_Alps_RK09L_Single_Vertical, F.Cu at (126.9, 77.0)
- added RV3: 5K, Potentiometer_THT:Potentiometer_Alps_RK09L_Single_Vertical, F.Cu at (127.3, 99.3)
- added RV4: 5K, Potentiometer_THT:Potentiometer_Alps_RK09L_Single_Vertical, F.Cu at (126.2, 124.3)
- added SW2: SW_SPST, Connector_PinHeader_2.54mm:PinHeader_1x02_P2.54mm_Vertical, F.Cu at (7.24, 84.1)
- added SW3: SW_SPST, Connector_PinHeader_2.54mm:PinHeader_1x02_P2.54mm_Vertical, F.Cu at (8.76, 106.6)
- added SW4: SW_SPST, Connector_PinHeader_2.54mm:PinHeader_1x02_P2.54mm_Vertical, F.Cu at (8.45, 129.5)
- C1, C10, C11, C12, C13, C14, C15, C16, C17, C2, C3, C4, C5, C7, C8, C9, D5, R1, R2, R3, R4, R5, R6, R7, R8, TP1, TP3, U1, U10, U2, U3, U4, U5, U6, U7, U8, U9: moved to B.Cu
- D1, D2, D3, D4: footprint LED_SMD:LED_0805_2012Metric_Pad1.15x1.40mm_HandSolder -> LED_THT:LED_D5.0mm
- J1, J2, J3, J4, J5, J6: moved to F.Cu
- SW1: value SW_DIP_x04 -> SW_SPST; footprint Button_Switch_SMD:SW_DIP_SPSTx04_Slide_6.7x11.72mm_W6.73mm_P2.54mm_LowProfile_JPin -> Connector_PinHeader_2.54mm:PinHeader_1x02_P2.54mm_Vertical
- moved D4 138.0 mm to (-5.84, 131.1)
- moved R4 131.2 mm to (1.65, 131.6)
- moved D3 119.0 mm to (-6.73, 106.7)
- moved R3 111.3 mm to (1.97, 107.7), turned to 90 degrees
- moved D2 101.3 mm to (-6.73, 81.9)
- moved R2 93.8 mm to (1.14, 83.4), turned to 90 degrees
- moved D1 87.4 mm to (-6.99, 56.9)
- moved R1 79.0 mm to (0.51, 57.5), turned to 90 degrees
- moved SW1 65.4 mm to (7.81, 58.5), turned to 180 degrees
- moved C10 14.2 mm to (190.5, 84.1)
- moved C11 13.0 mm to (182.2, 83.4)
- moved C3 12.8 mm to (196.8, 71.9)
- moved C9 9.14 mm to (190.5, 81.5)
- moved C5 7.75 mm to (207.6, 69.3)
- moved J4 6.99 mm to (54.0, 127.5)
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Connections:
- R1 pad 2: /BUFFER_SW4 -> /BUFFER_SW1
- R2 pad 2: /BUFFER_SW3 -> /BUFFER_SW2
- R3 pad 2: /BUFFER_SW2 -> /BUFFER_SW3
- R4 pad 2: /BUFFER_SW1 -> /BUFFER_SW4
- SW1 pad 2: +5V -> /BUFFER_SW1
- U1 pad 1: Net-(U1-Pad1) -> Net-(R20-Pad1)
- U1 pad 3: /SignalBuffer1/IN -> GNDS
- U1 pad 4: Net-(U1-Pad1) -> Net-(R15-Pad1)
- U2 pad 1: Net-(U2-Pad1) -> Net-(R18-Pad1)
- U2 pad 3: /SignalBuffer1/IN -> GNDS
- U2 pad 4: Net-(U2-Pad1) -> Net-(R13-Pad1)
- U3 pad 1: Net-(U3-Pad1) -> Net-(R16-Pad1)
- U3 pad 3: /SignalBuffer1/IN -> GNDS
- U3 pad 4: Net-(U3-Pad1) -> Net-(R11-Pad1)
- U4 pad 1: Net-(U4-Pad1) -> Net-(R12-Pad1)
- U4 pad 3: /SignalBuffer1/IN -> GNDS
- U4 pad 4: Net-(U4-Pad1) -> Net-(R10-Pad2)
- U5 pad 1: Net-(U1-Pad1) -> Net-(R20-Pad1)
- U6 pad 1: Net-(U2-Pad1) -> Net-(R18-Pad1)
- U7 pad 1: Net-(U3-Pad1) -> Net-(R16-Pad1)
- U8 pad 1: Net-(U4-Pad1) -> Net-(R12-Pad1)
Routing:
- net GNDS: track 7.62 -> 0.00 mm
- net +5V: track 7.62 -> 0.00 mm
- net /BUFFER_SW4: track 4.50 -> 0.00 mm
- net /BUFFER_SW3: track 4.50 -> 0.00 mm
- net /BUFFER_SW2: track 4.50 -> 0.00 mm
- net /BUFFER_SW1: track 4.50 -> 0.00 mm
- net Net-(D4-Pad2): track 2.40 -> 0.00 mm
- net Net-(D3-Pad2): track 2.40 -> 0.00 mm
- net Net-(D2-Pad2): track 2.40 -> 0.00 mm
- net Net-(D1-Pad2): track 2.40 -> 0.00 mm

Commit message: SOT23 REVA draft layout completed
Parts:
- removed TP1, TP3: TestPoint, TestPoint:TestPoint_Pad_1.0x1.0mm
- C1, C10, C11, C2, C3, C8, C9: footprint Capacitor_SMD:C_0402_1005Metric -> Capacitor_SMD:C_0805_2012Metric_Pad1.15x1.40mm_HandSolder
- J1, J2, J3, J4, J5, J6: moved to B.Cu
- R8: footprint Resistor_SMD:R_0402_1005Metric -> Resistor_SMD:R_0805_2012Metric_Pad1.15x1.40mm_HandSolder
- SW1, SW2, SW3, SW4: value SW_SPST -> SW_SPDT; footprint Connector_PinHeader_2.54mm:PinHeader_1x02_P2.54mm_Vertical -> RS_Switches:SPDT_Slide_Switch_Latching_Vertical_THT_8x9.3mm_734-7303
- moved J6 195.9 mm to (35.6, 113.3), turned to 0 degrees
- moved D5 180.5 mm to (41.3, 116.8)
- moved C5 171.7 mm to (41.3, 111.8)
- moved U9 159.8 mm to (48.3, 116.8)
- moved C1 155.5 mm to (53.3, 116.8), turned to 90 degrees
- moved C8 153.1 mm to (48.3, 111.8), turned to 0 degrees
- moved U10 143.5 mm to (58.4, 113.0), turned to 90 degrees
- moved C2 133.8 mm to (58.4, 108.0), turned to 0 degrees
- moved C3 133.8 mm to (68.1, 108.2), turned to 0 degrees
- moved C10 132.4 mm to (62.5, 117.9), turned to 0 degrees
- moved C9 129.4 mm to (66.0, 116.8), turned to 270 degrees
- moved R8 120.6 mm to (67.9, 111.8), turned to 0 degrees
- moved R7 117.9 mm to (81.8, 114.3), turned to 270 degrees
- moved R6 117.7 mm to (76.7, 116.8), turned to 90 degrees
- moved C11 117.3 mm to (69.8, 116.8), turned to 270 degrees
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Connections:
- C3 pad 1: -5V -> /PowerSupply/-5VOUT
- C9 pad 1: Net-(C9-Pad1) -> /PowerSupply/-5VOUT
- R1 pad 2: /BUFFER_SW1 -> /SignalBuffer1/BUFFER_SW1
- R2 pad 2: /BUFFER_SW2 -> /SignalBuffer2/BUFFER_SW1
- R3 pad 2: /BUFFER_SW3 -> /SignalBuffer3/BUFFER_SW1
- R4 pad 2: /BUFFER_SW4 -> /SignalBuffer4/BUFFER_SW1
- R8 pad 1: Net-(C9-Pad1) -> /PowerSupply/-5VOUT
- SW1 pad 1: +5V -> Net-(SW1-Pad1)
- SW1 pad 2: /BUFFER_SW1 -> +5V
- SW2 pad 1: +5V -> Net-(SW2-Pad1)
- SW2 pad 2: /BUFFER_SW2 -> +5V
- SW3 pad 1: +5V -> Net-(SW3-Pad1)
- SW3 pad 2: /BUFFER_SW3 -> +5V
- SW4 pad 1: +5V -> Net-(SW4-Pad1)
- SW4 pad 2: /BUFFER_SW4 -> +5V
- U10 pad 1: Net-(C9-Pad1) -> /PowerSupply/-5VOUT
- U5 pad 3: /BUFFER_SW1 -> /SignalBuffer1/BUFFER_SW1
- U6 pad 3: /BUFFER_SW2 -> /SignalBuffer2/BUFFER_SW1
- U7 pad 3: /BUFFER_SW3 -> /SignalBuffer3/BUFFER_SW1
- U8 pad 3: /BUFFER_SW4 -> /SignalBuffer4/BUFFER_SW1
Routing:
- net +5V: track 0.00 -> 240.8 mm, vias 0 -> 5
- net /SignalBuffer1/IN: track 0.00 -> 227.4 mm
- net -5V: track 0.00 -> 194.7 mm, vias 0 -> 5
- net GNDS: track 0.00 -> 149.4 mm, vias 0 -> 12
- net /SignalBuffer4/BUFFER_SW1: track 0.00 -> 36.0 mm
- net /SignalBuffer3/BUFFER_SW1: track 0.00 -> 35.8 mm
- net /SignalBuffer2/BUFFER_SW1: track 0.00 -> 35.7 mm
- net /SignalBuffer1/BUFFER_SW1: track 0.00 -> 34.5 mm
- net Net-(J5-Pad1): track 0.00 -> 21.7 mm
- net Net-(R18-Pad1): track 0.00 -> 19.2 mm
- net Net-(R16-Pad1): track 0.00 -> 18.7 mm
- net Net-(R12-Pad1): track 0.00 -> 18.7 mm
- net Net-(R20-Pad1): track 0.00 -> 17.9 mm
- net Net-(R10-Pad1): track 0.00 -> 17.6 mm
- net Net-(R19-Pad1): track 0.00 -> 17.5 mm
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- added copper zone on F.Cu, net GNDS
Other:
- board outline added: 94 x 91.4 mm
- net class Default: clearance 0.2 -> 0.127; trace_width 0.25 -> 0.127; via_dia 0.8 -> 0.45; via_drill 0.4 -> 0.2
- rule trace_clearance: 0.2 -> 0.127
- rule trace_min: 0.2 -> 0.127
- rule via_min_drill: 0.3 -> 0.2
- rule via_min_size: 0.4 -> 0.45

Commit message: updated SOT23 design layout outline to use 1590BB
Parts:
- moved J5 148.3 mm to (252.1, 102.9)
- moved RV4 133.5 mm to (165.0, 80.3)
- moved C16 133.3 mm to (169.0, 59.3)
- moved C17 133.3 mm to (169.0, 51.6)
- moved D4 133.3 mm to (164.8, 74.5)
- moved J4 133.3 mm to (167.4, 35.2)
- moved R10 133.3 mm to (173.2, 68.5)
- moved R12 133.3 mm to (175.3, 68.5)
- moved R4 133.3 mm to (162.3, 69.5)
- moved R9 133.3 mm to (171.2, 68.5)
- moved SW4 133.3 mm to (163.3, 57.3)
- moved U4 133.3 mm to (172.8, 59.3)
- moved U8 133.3 mm to (172.8, 51.6)
- moved RV1 131.0 mm to (232.9, 80.3)
- moved RV2 131.0 mm to (210.1, 80.3)
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Routing:
- net Net-(J5-Pad1): track 21.7 -> 49.0 mm
- net GNDS: track 149.4 -> 168.6 mm
- net /SignalBuffer1/IN: track 227.4 -> 220.9 mm
- net /PowerSupply/+9V_IN: track 13.5 -> 18.2 mm
- net Net-(R19-Pad1): track 17.5 -> 18.6 mm
- net Net-(R12-Pad2): track 14.9 -> 16.1 mm
- net /PowerSupply/-5VOUT: track 16.9 -> 15.9 mm
- net Net-(R18-Pad2): track 14.4 -> 15.4 mm
- net Net-(R16-Pad2): track 14.4 -> 15.4 mm
- net Net-(R10-Pad1): track 17.6 -> 18.5 mm
- net Net-(R14-Pad1): track 16.9 -> 17.7 mm
- net Net-(R20-Pad2): track 15.0 -> 15.7 mm
- net /PowerSupply/+9V_POL: track 9.95 -> 9.19 mm
- net Net-(R17-Pad1): track 16.9 -> 17.7 mm
- net Net-(C2-Pad2): track 3.76 -> 3.09 mm
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Other:
- board size 94 x 91.4 mm -> 124 x 100.8 mm
- board text added: "Active 4-Way Splitter Hammond 1590BB"

Commit message: Completed RevA layout
Parts:
- removed R13, R15: 2K2, Resistor_SMD:R_0805_2012Metric_Pad1.15x1.40mm_HandSolder
- removed R14, R16, R17, R18, R19, R20: 100R, Resistor_SMD:R_0805_2012Metric_Pad1.15x1.40mm_HandSolder
- removed SW1, SW2, SW3, SW4: SW_SPDT, RS_Switches:SPDT_Slide_Switch_Latching_Vertical_THT_8x9.3mm_734-7303
- removed U5, U6, U7, U8: DG468DV_T1_E3, Package_SO:TSOP-6_1.65x3.05mm_P0.95mm
- added C18: 1uF, Capacitor_SMD:C_0805_2012Metric_Pad1.15x1.40mm_HandSolder, B.Cu at (165.7, 83.8)
- added C19: 1uF, Capacitor_SMD:C_0805_2012Metric_Pad1.15x1.40mm_HandSolder, B.Cu at (170.8, 65.4)
- added C20: 1uF, Capacitor_SMD:C_0805_2012Metric_Pad1.15x1.40mm_HandSolder, B.Cu at (168.3, 69.8)
- added C6: 1uF, Capacitor_SMD:C_0805_2012Metric_Pad1.15x1.40mm_HandSolder, B.Cu at (239.4, 65.4)
- added D6: 1N914, Diode_SMD:D_SMB_Handsoldering, B.Cu at (184.8, 67.3)
- added D7: LED, LED_THT:LED_D5.0mm, F.Cu at (190.0, 42.2)
- added D8: 1N914, Diode_SMD:D_SMB_Handsoldering, B.Cu at (161.9, 67.3)
- added D9: LED, LED_THT:LED_D5.0mm, F.Cu at (167.4, 42.2)
- C12, C13, C14, C15, C16, C17, C4, C7: value 100nF -> 1uF
- D1, D3: value LED -> 1N914; footprint LED_THT:LED_D5.0mm -> Diode_SMD:D_SMB_Handsoldering; moved to B.Cu
- D5: footprint Diode_SMD:D_SOD-123F -> Diode_SMD:D_SMB_Handsoldering
- R1, R3: value 1K -> 100R
- R10, R12: value 100R -> 100K
- R11, R9: value 2K2 -> 100R
- R2, R4: value 1K -> 100K
- RV1, RV2, RV3, RV4: value 5K -> 1K; footprint Potentiometer_THT:Potentiometer_Alps_RK09L_Single_Vertical -> Bourn_PTA_Slider:Slider_PTA4543_60MM
- U1, U2, U3, U4: value OPA842 -> TL074; footprint Package_TO_SOT_SMD:SOT-23-5 -> Package_SO:SOIC-14_3.9x8.7mm_P1.27mm
- moved D4 58.1 mm to (213.1, 42.2), turned to 270 degrees
- moved R4 53.6 mm to (215.9, 69.8), turned to 270 degrees
- moved D2 41.6 mm to (236.0, 42.2), turned to 270 degrees
- moved R3 38.3 mm to (214.0, 94.0), turned to 270 degrees
- moved R11 34.7 mm to (168.3, 94.0)
- moved R9 32.4 mm to (191.1, 94.0)
- moved C12 32.3 mm to (211.5, 83.8), turned to 270 degrees
- moved C15 32.3 mm to (188.6, 83.8), turned to 270 degrees
- moved C4 32.2 mm to (234.9, 83.8), turned to 270 degrees
- moved R2 32.0 mm to (239.4, 69.8), turned to 270 degrees
- moved C17 28.7 mm to (191.1, 69.8)
- moved C3 26.1 mm to (207.6, 118.7), turned to 270 degrees
- moved R1 25.6 mm to (237.5, 94.0), turned to 270 degrees
- moved C16 25.4 mm to (193.7, 65.4)
- moved C2 24.5 mm to (201.3, 109.9)
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Connections:
- C13 pad 1: +5V -> -5V
- C14 pad 1: +5V -> Net-(C14-Pad1)
- C16 pad 1: +5V -> -5V
- C17 pad 1: +5V -> Net-(C17-Pad1)
- C7 pad 1: +5V -> Net-(C7-Pad1)
- D1 pad 1: GNDS -> Net-(C7-Pad1)
- D3 pad 1: GNDS -> Net-(C14-Pad1)
- J1 pad 1: /SignalBuffer1/OUT -> /GainAndPeakDetector1/SIGNAL_OUTPUT
- J2 pad 1: /SignalBuffer2/OUT -> /GainAndPeakDetector2/SIGNAL_OUTPUT
- J3 pad 1: /SignalBuffer3/OUT -> /GainAndPeakDetector3/SIGNAL_OUTPUT
- J4 pad 1: /SignalBuffer4/OUT -> /GainAndPeakDetector4/SIGNAL_OUTPUT
- R1 pad 1: Net-(D1-Pad2) -> Net-(R1-Pad1)
- R1 pad 2: /SignalBuffer1/BUFFER_SW1 -> /GainAndPeakDetector1/SIGNAL_INPUT
- R10 pad 1: Net-(R10-Pad1) -> GNDS
- R10 pad 2: Net-(R10-Pad2) -> Net-(C17-Pad1)
- R11 pad 2: /SignalBuffer1/IN -> /GainAndPeakDetector1/SIGNAL_INPUT
- R12 pad 1: Net-(R12-Pad1) -> GNDS
- R12 pad 2: Net-(R12-Pad2) -> Net-(C20-Pad1)
- R2 pad 1: Net-(D2-Pad2) -> GNDS
- R2 pad 2: /SignalBuffer2/BUFFER_SW1 -> Net-(C7-Pad1)
- R3 pad 1: Net-(D3-Pad2) -> Net-(R3-Pad1)
- R3 pad 2: /SignalBuffer3/BUFFER_SW1 -> /GainAndPeakDetector1/SIGNAL_INPUT
- R4 pad 1: Net-(D4-Pad2) -> GNDS
- R4 pad 2: /SignalBuffer4/BUFFER_SW1 -> Net-(C14-Pad1)
- R5 pad 1: /SignalBuffer1/IN -> /GainAndPeakDetector1/SIGNAL_INPUT
- R7 pad 1: /SignalBuffer1/IN -> /GainAndPeakDetector1/SIGNAL_INPUT
- R9 pad 1: Net-(R10-Pad2) -> Net-(R9-Pad1)
- R9 pad 2: /SignalBuffer1/IN -> /GainAndPeakDetector1/SIGNAL_INPUT
- RV1 pad 1: Net-(R19-Pad1) -> /GainAndPeakDetector1/SIGNAL_OUTPUT
- RV1 pad 2: Net-(R19-Pad1) -> /GainAndPeakDetector1/SIGNAL_OUTPUT
- RV1 pad 3: Net-(R20-Pad2) -> Net-(R1-Pad1)
- RV2 pad 1: Net-(R17-Pad1) -> /GainAndPeakDetector2/SIGNAL_OUTPUT
- RV2 pad 2: Net-(R17-Pad1) -> /GainAndPeakDetector2/SIGNAL_OUTPUT
- RV2 pad 3: Net-(R18-Pad2) -> Net-(R3-Pad1)
- RV3 pad 1: Net-(R14-Pad1) -> /GainAndPeakDetector3/SIGNAL_OUTPUT
- RV3 pad 2: Net-(R14-Pad1) -> /GainAndPeakDetector3/SIGNAL_OUTPUT
- RV3 pad 3: Net-(R16-Pad2) -> Net-(R9-Pad1)
- RV4 pad 1: Net-(R10-Pad1) -> /GainAndPeakDetector4/SIGNAL_OUTPUT
- RV4 pad 2: Net-(R10-Pad1) -> /GainAndPeakDetector4/SIGNAL_OUTPUT
- RV4 pad 3: Net-(R12-Pad2) -> Net-(R11-Pad1)
- U1 pad 1: Net-(R20-Pad1) -> /GainAndPeakDetector1/SIGNAL_OUTPUT
- U1 pad 2: -5V -> Net-(R1-Pad1)
- U1 pad 4: Net-(R15-Pad1) -> +5V
- U1 pad 5: +5V -> /GainAndPeakDetector1/SIGNAL_OUTPUT
- U2 pad 1: Net-(R18-Pad1) -> /GainAndPeakDetector2/SIGNAL_OUTPUT
- U2 pad 2: -5V -> Net-(R3-Pad1)
- U2 pad 4: Net-(R13-Pad1) -> +5V
- U2 pad 5: +5V -> /GainAndPeakDetector2/SIGNAL_OUTPUT
- U3 pad 1: Net-(R16-Pad1) -> /GainAndPeakDetector3/SIGNAL_OUTPUT
- U3 pad 2: -5V -> Net-(R9-Pad1)
- U3 pad 4: Net-(R11-Pad1) -> +5V
- U3 pad 5: +5V -> /GainAndPeakDetector3/SIGNAL_OUTPUT
- U4 pad 1: Net-(R12-Pad1) -> /GainAndPeakDetector4/SIGNAL_OUTPUT
- U4 pad 2: -5V -> Net-(R11-Pad1)
- U4 pad 4: Net-(R10-Pad2) -> +5V
- U4 pad 5: +5V -> /GainAndPeakDetector4/SIGNAL_OUTPUT
Routing:
- net /SignalBuffer1/IN: track 220.9 -> 0.00 mm
- net /GainAndPeakDetector1/SIGNAL_INPUT: track 0.00 -> 150.7 mm, vias 0 -> 2
- net /GainAndPeakDetector2/SIGNAL_OUTPUT: track 0.00 -> 60.0 mm
- net /GainAndPeakDetector1/SIGNAL_OUTPUT: track 0.00 -> 59.4 mm
- net /GainAndPeakDetector3/SIGNAL_OUTPUT: track 0.00 -> 57.8 mm
- net /GainAndPeakDetector4/SIGNAL_OUTPUT: track 0.00 -> 56.4 mm
- net +5V: track 241.4 -> 186.3 mm, vias 5 -> 4
- net Net-(D7-Pad2): track 0.00 -> 40.8 mm
- net Net-(D9-Pad2): track 0.00 -> 38.8 mm
- net Net-(R1-Pad1): track 0.00 -> 36.1 mm
- net /SignalBuffer4/BUFFER_SW1: track 36.0 -> 0.00 mm
- net /SignalBuffer3/BUFFER_SW1: track 35.8 -> 0.00 mm
- net Net-(R3-Pad1): track 0.00 -> 35.8 mm
- net /SignalBuffer2/BUFFER_SW1: track 35.7 -> 0.00 mm
- net Net-(R9-Pad1): track 0.00 -> 35.6 mm
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