File: ActiveSplitterPedal/RevB/SOIC14/ActiveSplitterPedal_SOIC14.kicad_pcb (KiCad board)
At the start: 2 copper layers, 112.5 x 86.4 mm, 78 parts, among them J1 MonoJack2Switch, J2 MonoJack2Switch, J3 MonoJack2Switch, J4 MonoJack2Switch, J5 MonoJack2Switch, J6 Barrel_Jack, U1 TL074, U2 TL074, U3 TL074, U4 TL074, U5 TPS60400, U6 TPS60400, U7 TPS60400, U8 TPS60400, U9 SE8250X2

Commit message: updated hw
completed revb layout
Parts:
- added R16: 1K, Resistor_SMD:R_0805_2012Metric_Pad1.15x1.40mm_HandSolder, B.Cu at (160.4, 102.7)
- added R17: 120K, Resistor_SMD:R_0805_2012Metric_Pad1.15x1.40mm_HandSolder, B.Cu at (164.2, 103.9)
- added R18: 1K, Resistor_SMD:R_0805_2012Metric_Pad1.15x1.40mm_HandSolder, B.Cu at (98.7, 102.9)
- added R19: 120K, Resistor_SMD:R_0805_2012Metric_Pad1.15x1.40mm_HandSolder, B.Cu at (102.4, 103.9)
- added R20: 1K, Resistor_SMD:R_0805_2012Metric_Pad1.15x1.40mm_HandSolder, B.Cu at (119.4, 102.9)
- added R21: 120K, Resistor_SMD:R_0805_2012Metric_Pad1.15x1.40mm_HandSolder, B.Cu at (123.1, 103.9)
- added R22: 1K, Resistor_SMD:R_0805_2012Metric_Pad1.15x1.40mm_HandSolder, B.Cu at (139.8, 102.7)
- added R23: 120K, Resistor_SMD:R_0805_2012Metric_Pad1.15x1.40mm_HandSolder, B.Cu at (143.6, 103.9)
- C11, C12, C13, C15, C16, C18, C19, C24, C28, C32, C4, C5, C6: value 1uF -> 100nF
- C8: value 10uF -> 1uF
- R1, R11, R3, R9: value 100R -> 560R
- R13, R14, R15, R8: value 100R -> 22R
- U5, U6, U7, U8: value TPS60400 -> TPS60403
- moved D1 17.3 mm to (154.4, 103.1), turned to 90 degrees
- moved D3 17.2 mm to (133.9, 103.1), turned to 90 degrees
- moved D8 17.1 mm to (177.9, 97.8)
- moved D6 17.1 mm to (113.1, 103.1), turned to 90 degrees
- moved R3 16.5 mm to (154.3, 128.9)
- moved R9 16.1 mm to (133.6, 128.9)
- moved R11 15.9 mm to (113.0, 128.9)
- moved R1 15.7 mm to (174.5, 128.9)
- moved C33 13.5 mm to (117.3, 87.6), turned to 270 degrees
- moved C35 13.1 mm to (158.9, 87.6), turned to 270 degrees
- moved C27 12.4 mm to (96.6, 80.0)
- moved C9 12.3 mm to (137.9, 80.0)
- moved C34 11.4 mm to (96.5, 87.6), turned to 270 degrees
- moved C3 11.2 mm to (137.9, 87.6), turned to 270 degrees
- moved C22 10.4 mm to (130.8, 80.0), turned to 270 degrees
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Connections:
- U1 pad 1: /GainAndPeakDetector1/SIGNAL_OUTPUT -> Net-(D8-Pad2)
- U1 pad 10: Net-(C7-Pad1) -> GNDS
- U1 pad 12: Net-(U1-Pad12) -> Net-(C7-Pad1)
- U1 pad 13: Net-(U1-Pad13) -> Net-(D2-Pad2)
- U1 pad 14: Net-(U1-Pad14) -> Net-(D2-Pad2)
- U1 pad 2: Net-(R1-Pad1) -> Net-(C7-Pad1)
- U1 pad 3: GNDS -> Net-(R17-Pad2)
- U1 pad 6: Net-(C7-Pad1) -> Net-(R16-Pad2)
- U1 pad 7: Net-(D8-Pad2) -> Net-(R17-Pad2)
- U1 pad 8: Net-(D2-Pad2) -> /GainAndPeakDetector1/SIGNAL_OUTPUT
- U1 pad 9: Net-(D2-Pad2) -> Net-(R1-Pad1)
- U2 pad 1: /GainAndPeakDetector2/SIGNAL_OUTPUT -> Net-(D1-Pad2)
- U2 pad 10: Net-(C14-Pad1) -> GNDS
- U2 pad 12: Net-(U2-Pad12) -> Net-(C14-Pad1)
- U2 pad 13: Net-(U2-Pad13) -> Net-(D4-Pad2)
- U2 pad 14: Net-(U2-Pad14) -> Net-(D4-Pad2)
- U2 pad 2: Net-(R3-Pad1) -> Net-(C14-Pad1)
- U2 pad 3: GNDS -> Net-(R23-Pad2)
- U2 pad 6: Net-(C14-Pad1) -> Net-(R22-Pad2)
- U2 pad 7: Net-(D1-Pad2) -> Net-(R23-Pad2)
- U2 pad 8: Net-(D4-Pad2) -> /GainAndPeakDetector2/SIGNAL_OUTPUT
- U2 pad 9: Net-(D4-Pad2) -> Net-(R3-Pad1)
- U3 pad 1: /GainAndPeakDetector3/SIGNAL_OUTPUT -> Net-(D3-Pad2)
- U3 pad 10: Net-(C17-Pad1) -> GNDS
- U3 pad 12: Net-(U3-Pad12) -> Net-(C17-Pad1)
- U3 pad 13: Net-(U3-Pad13) -> Net-(D7-Pad2)
- U3 pad 14: Net-(U3-Pad14) -> Net-(D7-Pad2)
- U3 pad 2: Net-(R9-Pad1) -> Net-(C17-Pad1)
- U3 pad 3: GNDS -> Net-(R21-Pad2)
- U3 pad 6: Net-(C17-Pad1) -> Net-(R20-Pad2)
- U3 pad 7: Net-(D3-Pad2) -> Net-(R21-Pad2)
- U3 pad 8: Net-(D7-Pad2) -> /GainAndPeakDetector3/SIGNAL_OUTPUT
- U3 pad 9: Net-(D7-Pad2) -> Net-(R9-Pad1)
- U4 pad 1: /GainAndPeakDetector4/SIGNAL_OUTPUT -> Net-(D6-Pad2)
- U4 pad 10: Net-(C20-Pad1) -> GNDS
- U4 pad 12: Net-(U4-Pad12) -> Net-(C20-Pad1)
- U4 pad 13: Net-(U4-Pad13) -> Net-(D9-Pad2)
- U4 pad 14: Net-(U4-Pad14) -> Net-(D9-Pad2)
- U4 pad 2: Net-(R11-Pad1) -> Net-(C20-Pad1)
- U4 pad 3: GNDS -> Net-(R19-Pad2)
- U4 pad 6: Net-(C20-Pad1) -> Net-(R18-Pad2)
- U4 pad 7: Net-(D6-Pad2) -> Net-(R19-Pad2)
- U4 pad 8: Net-(D9-Pad2) -> /GainAndPeakDetector4/SIGNAL_OUTPUT
- U4 pad 9: Net-(D9-Pad2) -> Net-(R11-Pad1)
Routing:
- net GNDS: track 149.6 -> 194.0 mm
- net Net-(R1-Pad1): track 91.6 -> 54.8 mm
- net Net-(R9-Pad1): track 91.0 -> 55.7 mm
- net Net-(R3-Pad1): track 90.0 -> 55.8 mm
- net Net-(R11-Pad1): track 91.2 -> 57.4 mm
- net /GainAndPeakDetector3/SIGNAL_OUTPUT: track 88.3 -> 64.5 mm
- net /GainAndPeakDetector2/SIGNAL_OUTPUT: track 85.1 -> 63.6 mm
- net /GainAndPeakDetector1/SIGNAL_OUTPUT: track 83.9 -> 63.4 mm
- net /GainAndPeakDetector4/SIGNAL_OUTPUT: track 85.1 -> 64.5 mm
- net /GainAndPeakDetector3/-5V_POL: track 31.9 -> 11.9 mm
- net /GainAndPeakDetector4/-5V_POL: track 31.5 -> 11.7 mm
- net /GainAndPeakDetector2/-5V_POL: track 31.5 -> 12.2 mm
- net /GainAndPeakDetector1/-5V_POL: track 30.8 -> 11.6 mm
- net Net-(R19-Pad2): track 0.00 -> 17.4 mm
- net Net-(R21-Pad2): track 0.00 -> 16.8 mm
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
Commit message: Completed Revb LAyout
Parts:
- added C36: 1pF, Capacitor_SMD:C_0805_2012Metric_Pad1.15x1.40mm_HandSolder, B.Cu at (120.0, 94.5)
- added C37: 1uF, Capacitor_SMD:C_Elec_4x5.8, B.Cu at (124.1, 118.6)
- added C38: 1pF, Capacitor_SMD:C_0805_2012Metric_Pad1.15x1.40mm_HandSolder, B.Cu at (140.5, 94.5)
- added C39: 1uF, Capacitor_SMD:C_Elec_4x5.8, B.Cu at (144.8, 118.6)
- added R24: 100R, Resistor_SMD:R_0805_2012Metric_Pad1.15x1.40mm_HandSolder, B.Cu at (118.6, 69.3)
- added R25: 220R, Resistor_SMD:R_0805_2012Metric_Pad1.15x1.40mm_HandSolder, B.Cu at (133.6, 70.6)
- added R26: 100R, Resistor_SMD:R_0805_2012Metric_Pad1.15x1.40mm_HandSolder, B.Cu at (139.4, 69.6)
- added R27: 220R, Resistor_SMD:R_0805_2012Metric_Pad1.15x1.40mm_HandSolder, B.Cu at (153.9, 70.6)
- C14, C20: footprint Capacitor_SMD:C_0805_2012Metric_Pad1.15x1.40mm_HandSolder -> Capacitor_SMD:C_Elec_4x5.8
- C17, C7: value 1uF -> 1pF
- D1, D3, D6, D8: footprint Diode_SMD:D_SMB_Handsoldering -> Diode_SMD:D_SOD-123F
- R10, R2: value 100K -> 100R
- R12, R4: value 100K -> 220R
- moved R10 38.9 mm to (97.5, 69.3), turned to 0 degrees
- moved C14 34.8 mm to (165.1, 118.6), turned to 180 degrees
- moved C20 31.3 mm to (103.8, 118.6), turned to 180 degrees
- moved C17 30.5 mm to (99.1, 94.5)
- moved R4 28.3 mm to (175.0, 70.6)
- moved R2 22.3 mm to (159.8, 69.5), turned to 0 degrees
- moved D8 20.6 mm to (165.4, 114.0), turned to 180 degrees
- moved R12 17.1 mm to (112.5, 70.6)
- moved D1 14.4 mm to (145.0, 114.0), turned to 180 degrees
- moved D3 14.4 mm to (124.5, 114.0), turned to 180 degrees
- moved D6 14.1 mm to (104.2, 114.0), turned to 180 degrees
- moved C7 11.1 mm to (161.0, 94.5)
- moved R22 6.99 mm to (140.0, 109.7)
- moved R18 6.87 mm to (99.1, 109.7)
- moved R20 6.86 mm to (119.4, 109.7)
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Connections:
- C17 pad 1: Net-(C17-Pad1) -> /GainAndPeakDetector4/SIGNAL_OUTPUT
- C17 pad 2: GNDS -> Net-(C17-Pad2)
- C7 pad 1: Net-(C7-Pad1) -> /GainAndPeakDetector1/SIGNAL_OUTPUT
- C7 pad 2: GNDS -> Net-(C7-Pad2)
- D1 pad 1: Net-(C14-Pad1) -> Net-(C39-Pad1)
- D3 pad 1: Net-(C17-Pad1) -> Net-(C37-Pad1)
- D8 pad 1: Net-(C7-Pad1) -> Net-(C14-Pad1)
- R1 pad 1: Net-(R1-Pad1) -> Net-(C7-Pad2)
- R10 pad 1: GNDS -> /GainAndPeakDetector4/SIGNAL_OUTPUT
- R10 pad 2: Net-(C17-Pad1) -> Net-(R10-Pad2)
- R11 pad 1: Net-(R11-Pad1) -> Net-(C17-Pad2)
- R12 pad 1: GNDS -> Net-(D9-Pad2)
- R12 pad 2: Net-(C20-Pad1) -> Net-(R12-Pad2)
- R2 pad 1: GNDS -> /GainAndPeakDetector1/SIGNAL_OUTPUT
- R2 pad 2: Net-(C7-Pad1) -> Net-(R2-Pad2)
- R4 pad 1: GNDS -> Net-(D2-Pad2)
- R4 pad 2: Net-(C14-Pad1) -> Net-(R4-Pad2)
- RV1 pad 1: /GainAndPeakDetector1/SIGNAL_OUTPUT -> Net-(R2-Pad2)
- RV1 pad 2: /GainAndPeakDetector1/SIGNAL_OUTPUT -> Net-(R2-Pad2)
- RV1 pad 3: Net-(R1-Pad1) -> Net-(C7-Pad2)
- RV2 pad 1: /GainAndPeakDetector2/SIGNAL_OUTPUT -> Net-(R26-Pad2)
- RV2 pad 2: /GainAndPeakDetector2/SIGNAL_OUTPUT -> Net-(R26-Pad2)
- RV3 pad 1: /GainAndPeakDetector3/SIGNAL_OUTPUT -> Net-(R24-Pad2)
- RV3 pad 2: /GainAndPeakDetector3/SIGNAL_OUTPUT -> Net-(R24-Pad2)
- RV4 pad 1: /GainAndPeakDetector4/SIGNAL_OUTPUT -> Net-(R10-Pad2)
- RV4 pad 2: /GainAndPeakDetector4/SIGNAL_OUTPUT -> Net-(R10-Pad2)
- RV4 pad 3: Net-(R11-Pad1) -> Net-(C17-Pad2)
- U1 pad 1: Net-(D8-Pad2) -> Net-(C14-Pad1)
- U1 pad 12: Net-(C7-Pad1) -> Net-(C14-Pad1)
- U1 pad 13: Net-(D2-Pad2) -> Net-(R4-Pad2)
- U1 pad 14: Net-(D2-Pad2) -> Net-(R4-Pad2)
- U1 pad 2: Net-(C7-Pad1) -> Net-(D8-Pad2)
- U1 pad 9: Net-(R1-Pad1) -> Net-(C7-Pad2)
- U2 pad 1: Net-(D1-Pad2) -> Net-(C39-Pad1)
- U2 pad 12: Net-(C14-Pad1) -> Net-(C39-Pad1)
- U2 pad 13: Net-(D4-Pad2) -> Net-(R27-Pad2)
- U2 pad 14: Net-(D4-Pad2) -> Net-(R27-Pad2)
- U2 pad 2: Net-(C14-Pad1) -> Net-(D1-Pad2)
- U3 pad 1: Net-(D3-Pad2) -> Net-(C37-Pad1)
- U3 pad 12: Net-(C17-Pad1) -> Net-(C37-Pad1)
- U3 pad 13: Net-(D7-Pad2) -> Net-(R25-Pad2)
- U3 pad 14: Net-(D7-Pad2) -> Net-(R25-Pad2)
- U3 pad 2: Net-(C17-Pad1) -> Net-(D3-Pad2)
- U4 pad 1: Net-(D6-Pad2) -> Net-(C20-Pad1)
- U4 pad 13: Net-(D9-Pad2) -> Net-(R12-Pad2)
- U4 pad 14: Net-(D9-Pad2) -> Net-(R12-Pad2)
- U4 pad 2: Net-(C20-Pad1) -> Net-(D6-Pad2)
- U4 pad 9: Net-(R11-Pad1) -> Net-(C17-Pad2)
Routing:
- net Net-(C17-Pad2): track 0.00 -> 58.3 mm, vias 0 -> 2
- net Net-(R11-Pad1): track 57.4 -> 0.00 mm, vias 2 -> 0
- net Net-(C7-Pad2): track 0.00 -> 56.8 mm, vias 0 -> 2
- net Net-(R1-Pad1): track 54.8 -> 0.00 mm, vias 2 -> 0
- net +5V: track 284.2 -> 253.5 mm, vias 13 -> 9
- net Net-(C37-Pad1): track 0.00 -> 29.8 mm
- net Net-(C39-Pad1): track 0.00 -> 28.1 mm
- net Net-(D7-Pad2): track 54.1 -> 26.6 mm
- net Net-(R4-Pad2): track 0.00 -> 27.2 mm
- net Net-(D9-Pad2): track 53.3 -> 26.2 mm
- net Net-(R25-Pad2): track 0.00 -> 27.1 mm
- net Net-(R27-Pad2): track 0.00 -> 27.0 mm
- net Net-(R12-Pad2): track 0.00 -> 26.9 mm
- net Net-(D2-Pad2): track 53.2 -> 26.5 mm
- net Net-(D4-Pad2): track 52.4 -> 26.2 mm
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