File: ActiveSplitterPedal/RevB/SOIC14/InvGainAndPeakDetector.sch (KiCad schematic (older format))
At the start: 18 parts, among them U1 TL074, U5 TPS60403

Commit message: updated hw
completed revb layout
Connections:
- net GNDS: now also U1.10 (+); no longer U1.3 (+)
- net SIGNAL_OUTPUT: now also U1.5 (+), U1.8; no longer U1.1, U1.12 (+)
- net at R1.1, RV1.3: now also U1.9 (-); no longer U1.2 (-)
- net at C7.1, D8.1 (K), R2.2: now also U1.12 (+), U1.2 (-); no longer U1.10 (+), U1.6 (-)
- net at D8.2 (A): now also U1.1; no longer U1.7
- net at R16.2, R17.1: now also U1.6 (-); no longer U1.13 (-)
- new net: R17.2, U1.3 (+), U1.7
- new net: D2.2 (A), U1.13 (-), U1.14
Other:
- moved on the sheet: U4A, U4B, U4C, U4D
Changed lines of the file:
@@
 $Descr A4 11693 8268
 encoding utf-8
-Sheet 3 6
+Sheet 4 6
 Title ""
 Date ""
@@
 L Amplifier_Operational:TL074 U1
 U 1 1 5F3F57C8
-P 2500 2550
+P 6450 3100
 AR Path="/5F3F1F31/5F3F57C8" Ref="U1"  Part="1"
 AR Path="/5F512144/5F3F57C8" Ref="U2"  Part="1"
 AR Path="/5F515E89/5F3F57C8" Ref="U3"  Part="1"
 AR Path="/5F519B24/5F3F57C8" Ref="U4"  Part="1"
-F 0 "U1" H 2550 2775 50  0000 C CNN
-F 1 "TL074" H 2550 2875 50  0000 C CNN
-F 2 "Package_SO:SOIC-14_3.9x8.7mm_P1.27mm" H 2450 2650 50  0001 C CNN
-F 3 "http://www.ti.com/lit/ds/symlink/tl071.pdf" H 2550 2750 50  0001 C CNN
-	1    2500 2550
-	1    0    0    1
+F 0 "U4" H 6500 3325 50  0000 C CNN
+F 1 "TL074" H 6500 3425 50  0000 C CNN
+F 2 "Package_SO:SOIC-14_3.9x8.7mm_P1.27mm" H 6400 3200 50  0001 C CNN
+F 3 "http://www.ti.com/lit/ds/symlink/tl071.pdf" H 6500 3300 50  0001 C CNN
+	1    6450 3100
+	1    0    0    -1
 $EndComp
 $Comp
 L Amplifier_Operational:TL074 U1
 U 2 1 5F3F63C2
-P 6450 3100
+P 4900 3000
 AR Path="/5F3F1F31/5F3F63C2" Ref="U1"  Part="2"
 AR Path="/5F512144/5F3F63C2" Ref="U2"  Part="2"
 AR Path="/5F515E89/5F3F63C2" Ref="U3"  Part="2"
 AR Path="/5F519B24/5F3F63C2" Ref="U4"  Part="2"
-F 0 "U1" H 6450 2875 50  0000 C CNN
-F 1 "TL074" H 6450 2775 50  0000 C CNN
-F 2 "Package_SO:SOIC-14_3.9x8.7mm_P1.27mm" H 6400 3200 50  0001 C CNN
-F 3 "http://www.ti.com/lit/ds/symlink/tl071.pdf" H 6500 3300 50  0001 C CNN
-	2    6450 3100
+F 0 "U4" H 4900 2775 50  0000 C CNN
+F 1 "TL074" H 4900 2675 50  0000 C CNN
+F 2 "Package_SO:SOIC-14_3.9x8.7mm_P1.27mm" H 4850 3100 50  0001 C CNN
+F 3 "http://www.ti.com/lit/ds/symlink/tl071.pdf" H 4950 3200 50  0001 C CNN
+	2    4900 3000
 	1    0    0    -1
 $EndComp
@@
 L Amplifier_Operational:TL074 U1
 U 3 1 5F3F80E5
-P 9600 3200
+P 2500 2550
 AR Path="/5F3F1F31/5F3F80E5" Ref="U1"  Part="3"
 AR Path="/5F512144/5F3F80E5" Ref="U2"  Part="3"
 AR Path="/5F515E89/5F3F80E5" Ref="U3"  Part="3"
 AR Path="/5F519B24/5F3F80E5" Ref="U4"  Part="3"
-F 0 "U1" H 9600 3567 50  0000 C CNN
-F 1 "TL074" H 9600 3476 50  0000 C CNN
-F 2 "Package_SO:SOIC-14_3.9x8.7mm_P1.27mm" H 9550 3300 50  0001 C CNN
-F 3 "http://www.ti.com/lit/ds/symlink/tl071.pdf" H 9650 3400 50  0001 C CNN
-	3    9600 3200
-	1    0    0    -1
+F 0 "U4" H 2500 2917 50  0000 C CNN
+F 1 "TL074" H 2500 2826 50  0000 C CNN
+F 2 "Package_SO:SOIC-14_3.9x8.7mm_P1.27mm" H 2450 2650 50  0001 C CNN
+F 3 "http://www.ti.com/lit/ds/symlink/tl071.pdf" H 2550 2750 50  0001 C CNN
+	3    2500 2550
+	1    0    0    1
 $EndComp
 $Comp
 L Amplifier_Operational:TL074 U1
 U 4 1 5F3F8AC2
-P 4900 3000
+P 9600 3200
 AR Path="/5F3F1F31/5F3F8AC2" Ref="U1"  Part="4"
 AR Path="/5F512144/5F3F8AC2" Ref="U2"  Part="4"
 AR Path="/5F515E89/5F3F8AC2" Ref="U3"  Part="4"
 AR Path="/5F519B24/5F3F8AC2" Ref="U4"  Part="4"
-F 0 "U1" H 4900 3367 50  0000 C CNN
-F 1 "TL074" H 4900 3276 50  0000 C CNN
-F 2 "Package_SO:SOIC-14_3.9x8.7mm_P1.27mm" H 4850 3100 50  0001 C CNN
-F 3 "http://www.ti.com/lit/ds/symlink/tl071.pdf" H 4950 3200 50  0001 C CNN
-	4    4900 3000
+F 0 "U4" H 9600 3567 50  0000 C CNN
+F 1 "TL074" H 9600 3476 50  0000 C CNN
+F 2 "Package_SO:SOIC-14_3.9x8.7mm_P1.27mm" H 9550 3300 50  0001 C CNN
+F 3 "http://www.ti.com/lit/ds/symlink/tl071.pdf" H 9650 3400 50  0001 C CNN
+	4    9600 3200
 	1    0    0    -1
 $EndComp
@@
 AR Path="/5F515E89/5F3F9579" Ref="U3"  Part="5"
 AR Path="/5F519B24/5F3F9579" Ref="U4"  Part="5"
-F 0 "U1" H 8850 5425 50  0000 R CNN
+F 0 "U4" H 8850 5425 50  0000 R CNN
 F 1 "TL074" H 8900 5325 50  0000 R CNN
 F 2 "Package_SO:SOIC-14_3.9x8.7mm_P1.27mm" H 8650 5475 50  0001 C CNN
@@
 AR Path="/5F515E89/5F415E0A" Ref="R9"  Part="1"
 AR Path="/5F519B24/5F415E0A" Ref="R11"  Part="1"
-F 0 "R1" V 1293 2450 50  0000 C CNN
+F 0 "R11" V 1293 2450 50  0000 C CNN
 F 1 "560R" V 1384 2450 50  0000 C CNN
 F 2 "Resistor_SMD:R_0805_2012Metric_Pad1.15x1.40mm_HandSolder" V 1430 2450 50  0001 C CNN
@@
 AR Path="/5F515E89/5F4179D2" Ref="RV3"  Part="1"
 AR Path="/5F519B24/5F4179D2" Ref="RV4"  Part="1"
-F 0 "RV1" V 3275 1950 50  0000 C CNN
+F 0 "RV4" V 3275 1950 50  0000 C CNN
 F 1 "1K" V 3175 1950 50  0000 C CNN
 F 2 "Bourn_PTA_Slider:Slider_PTA4543_60MM" H 2700 1950 50  0001 C CNN
@@
 AR Path="/5F515E89/5F431259" Ref="R10"  Part="1"
 AR Path="/5F519B24/5F431259" Ref="R12"  Part="1"
-F 0 "R2" H 7880 3604 50  0000 R CNN
+F 0 "R12" H 7880 3604 50  0000 R CNN
 F 1 "100K" H 7880 3695 50  0000 R CNN
 F 2 "Resistor_SMD:R_0805_2012Metric_Pad1.15x1.40mm_HandSolder" V 7880 3650 50  0001 C CNN
@@
 AR Path="/5F515E89/5F43779A" Ref="C17"  Part="1"
 AR Path="/5F519B24/5F43779A" Ref="C20"  Part="1"
-F 0 "C7" H 8615 3696 50  0000 L CNN
+F 0 "C20" H 8615 3696 50  0000 L CNN
 F 1 "1uF" H 8615 3605 50  0000 L CNN
 F 2 "Capacitor_SMD:C_0805_2012Metric_Pad1.15x1.40mm_HandSolder" H 8538 3500 50  0001 C CNN
@@
 AR Path="/5F515E89/5F44F4A6" Ref="C16"  Part="1"
 AR Path="/5F519B24/5F44F4A6" Ref="C19"  Part="1"
-F 0 "C6" H 9415 6071 50  0000 L CNN
+F 0 "C19" H 9415 6071 50  0000 L CNN
 F 1 "100nF" H 9415 5980 50  0000 L CNN
 F 2 "Capacitor_SMD:C_0805_2012Metric_Pad1.15x1.40mm_HandSolder" H 9338 5875 50  0001 C CNN
@@
 AR Path="/5F515E89/5F45B6FE" Ref="C15"  Part="1"
 AR Path="/5F519B24/5F45B6FE" Ref="C18"  Part="1"
-F 0 "C4" H 9415 5296 50  0000 L CNN
+F 0 "C18" H 9415 5296 50  0000 L CNN
 F 1 "100nF" H 9415 5205 50  0000 L CNN
 F 2 "Capacitor_SMD:C_0805_2012Metric_Pad1.15x1.40mm_HandSolder" H 9338 5100 50  0001 C CNN
@@
 AR Path="/5F515E89/5F4B9375" Ref="D7"  Part="1"
 AR Path="/5F519B24/5F4B9375" Ref="D9"  Part="1"
-F 0 "D2" V 10589 3532 50  0000 R CNN
+F 0 "D9" V 10589 3532 50  0000 R CNN
 F 1 "LED" V 10498 3532 50  0000 R CNN
 F 2 "LED_THT:LED_D5.0mm" H 10550 3650 50  0001 C CNN
@@
 AR Path="/5F515E89/5F3FDBB2" Ref="D3"  Part="1"
 AR Path="/5F519B24/5F3FDBB2" Ref="D6"  Part="1"
-F 0 "D8" H 7050 2883 50  0000 C CNN
+F 0 "D6" H 7050 2883 50  0000 C CNN
 F 1 "D_Schottky" H 7050 2974 50  0000 C CNN
 F 2 "Diode_SMD:D_SMB_Handsoldering" H 7050 3100 50  0001 C CNN
@@
 AR Path="/5F519B24/5F457D40" Ref="C34"  Part="1"
 AR Path="/5F3F1F31/5F457D40" Ref="C35"  Part="1"
-F 0 "C35" H 10340 5571 50  0000 L CNN
+F 0 "C34" H 10340 5571 50  0000 L CNN
 F 1 "100nF" H 10340 5480 50  0000 L CNN
 F 2 "Capacitor_SMD:C_0805_2012Metric_Pad1.15x1.40mm_HandSolder" H 10263 5375 50  0001 C CNN
@@
 AR Path="/5F519B24/5F414AF0" Ref="R14"  Part="1"
 AR Path="/5F3F1F31/5F414AF0" Ref="R15"  Part="1"
-F 0 "R15" V 5100 5975 50  0000 L CNN
+F 0 "R14" V 5100 5975 50  0000 L CNN
 F 1 "22R" V 5025 5875 50  0000 L CNN
 F 2 "Resistor_SMD:R_0805_2012Metric_Pad1.15x1.40mm_HandSolder" V 4855 5975 50  0001 C CNN
@@
 AR Path="/5F519B24/5F414AE2" Ref="C28"  Part="1"
 AR Path="/5F3F1F31/5F414AE2" Ref="C32"  Part="1"
-F 0 "C32" H 5440 6321 50  0000 L CNN
+F 0 "C28" H 5440 6321 50  0000 L CNN
 F 1 "100nF" H 5440 6230 50  0000 L CNN
 F 2 "Capacitor_SMD:C_0805_2012Metric_Pad1.15x1.40mm_HandSolder" H 5363 6125 50  0001 C CNN
@@
 AR Path="/5F519B24/5F414AD2" Ref="C27"  Part="1"
 AR Path="/5F3F1F31/5F414AD2" Ref="C31"  Part="1"
-F 0 "C31" H 4365 6321 50  0000 L CNN
+F 0 "C27" H 4365 6321 50  0000 L CNN
 F 1 "1uF" H 4365 6230 50  0000 L CNN
 F 2 "Capacitor_SMD:C_0805_2012Metric_Pad1.15x1.40mm_HandSolder" H 4288 6125 50  0001 C CNN
@@
 AR Path="/5F519B24/5F414AC2" Ref="C25"  Part="1"
 AR Path="/5F3F1F31/5F414AC2" Ref="C29"  Part="1"
-F 0 "C29" H 1575 6325 50  0000 L CNN
+F 0 "C25" H 1575 6325 50  0000 L CNN
 F 1 "1uF" H 1575 6225 50  0000 L CNN
 F 2 "Capacitor_SMD:C_0805_2012Metric_Pad1.15x1.40mm_HandSolder" H 1888 6125 50  0001 C CNN
@@
 AR Path="/5F519B24/5F414AB4" Ref="U7"  Part="1"
 AR Path="/5F3F1F31/5F414AB4" Ref="U8"  Part="1"
-F 0 "U8" H 2975 6830 50  0000 C CNN
+F 0 "U7" H 2975 6830 50  0000 C CNN
 F 1 "TPS60403" H 2975 6739 50  0000 C CNN
 F 2 "Package_TO_SOT_SMD:SOT-23-5_HandSoldering" H 2975 6648 50  0000 C CNN
@@
 AR Path="/5F519B24/5F414AAD" Ref="C26"  Part="1"
 AR Path="/5F3F1F31/5F414AAD" Ref="C30"  Part="1"
-F 0 "C30" H 2340 6321 50  0000 L CNN
+F 0 "C26" H 2340 6321 50  0000 L CNN
 F 1 "1uF" H 2340 6230 50  0000 L CNN
 F 2 "Capacitor_SMD:C_0805_2012Metric_Pad1.15x1.40mm_HandSolder" H 2263 6125 50  0001 C CNN
@@
 AR Path="/5F515E89/5F57D775" Ref="R21"  Part="1"
 AR Path="/5F519B24/5F57D775" Ref="R19"  Part="1"
-F 0 "R17" V 4950 3550 50  0000 R CNN
+F 0 "R19" V 4950 3550 50  0000 R CNN
 F 1 "120K" V 4750 3600 50  0000 R CNN
 F 2 "Resistor_SMD:R_0805_2012Metric_Pad1.15x1.40mm_HandSolder" V 4780 3500 50  0001 C CNN
@@
 AR Path="/5F515E89/5F58191C" Ref="R20"  Part="1"
 AR Path="/5F519B24/5F58191C" Ref="R18"  Part="1"
-F 0 "R16" H 4650 3700 50  0000 R CNN
+F 0 "R18" H 4650 3700 50  0000 R CNN
 F 1 "1K" H 4650 3800 50  0000 R CNN
 F 2 "Resistor_SMD:R_0805_2012Metric_Pad1.15x1.40mm_HandSolder" V 4380 3750 50  0001 C CNN

Commit message: Completed Revb LAyout
Parts:
- added C14: 1uF, Capacitor_SMD:C_Elec_4x5.8, symbol Device:CP
- added R4: 220R, Resistor_SMD:R_0805_2012Metric_Pad1.15x1.40mm_HandSolder, symbol Device:R
- C7: value 1uF -> 1pF
- D8: footprint Diode_SMD:D_SMB_Handsoldering -> Diode_SMD:D_SOD-123F
- R2: value 100K -> 100R
Connections:
- net GNDS: now also C14.2; no longer C7.2, R2.1
- net SIGNAL_OUTPUT: now also C7.1, R2.1; no longer RV1.1, RV1.2
- net at U1.1: now also D8.1 (K), U1.12 (+), C14.1; no longer D8.2 (A)
- net at R1.1, RV1.3, U1.9 (-): now also C7.2
- net at U1.13 (-), U1.14: now also R4.2; no longer D2.2 (A)
- new net: D8.2 (A), U1.2 (-)
- new net: R2.2, RV1.1, RV1.2
- new net: D2.2 (A), R4.1
Other:
- note added: "if using RVf=10K use Rin=5K6"
- note removed: "if using RV1=10K use R1=5K6"
- moved on the sheet: D2, D8, R16, RV1, U1D
