File: ActiveSplitterPedal/RevD/SOIC14/ActiveSplitterPedal_SOIC14.kicad_pcb (KiCad board)
At the start: 2 copper layers, 112.5 x 86.4 mm, 81 parts, among them J1 MonoJack2Switch, J2 Barrel_Jack, J3 MonoJack2Switch, J4 MonoJack2Switch, J5 MonoJack2Switch, J6 MonoJack2Switch, U1 MCP1700-5002E_SOT23, U11 TL072, U12 TL074, U14 ISA0505, U15 MCP1754S-3302xCB, U16 TC593002ECB, U2 TL072, U3 TL074, U5 TL072, U6 TL074, U8 TL072, U9 TL074

Commit message: updated
Parts:
- U1: value MCP1700-5002E_SOT23 -> SE8250X2
Other:
- board text added: "MIrror, Negative for F.Cu layer MIrror, Negative for B.Cu layer"
- board text removed: "Do not mirror if etching."
